File: RHF0M301-PI-Adapter.brd (EAGLE design)
At the start: 65 x 56 mm, 14 parts, among them J1 USB Micro Type B, U1 NEO-M8, U2 RHF0M301, X2 RASPI_BOARD_B+_H

Commit message: updated v1.1
Parts:
- added R2: 22, #afb-Passives:0603_MP
- C6: value 220uF 6V -> 10nF; device microbuilder:EIA6032-28/C-R -> #afb-Passives:0603_MP
- moved C6 17.1 mm to (56.0, 30.2), turned to 90 degrees
- moved C3 5.08 mm to (50.8, 14.0)
Connections:
- new net N$1: C6.1, R2.2, U2.14
- net GND: now also C6.2, J1.M1, J1.M2, J1.M3, J1.M4, J1.M5, J1.M6; no longer C6.-
- net RST: now also R2.1, X2.22; no longer U2.14, X2.26
- net VCC: no longer C6.+
Routing:
- net GND: track 186.9 -> 180.3 mm, vias 36 -> 39
- net N$1: track 0.00 -> 4.47 mm
- net V+: track 13.2 -> 14.5 mm
- net RST: track 44.5 -> 43.3 mm, vias 1 -> 0
- added copper zone on layer 1, net V+
Other:
- board text added: "RisingHF RHF0M301 Raspberry Pi Adapter v1.1"
- board text removed: "RisingHF RHF0301 Raspberry Pi Adapter v1.0"
